File: sensors.sch (KiCad schematic (older format))
At the start: 14 parts, among them U10 HMC5883L, U11 H3LIS331DL, U8 MS5611-01BA, U9 MPU6000

Commit message: changed sensors power supply (VCC_IO = VCC_A)
- all sensors and the eeprom are now powered by VCC_A
- internal I2C pullups to VCC_A
Reason: MS5611-01BA, HMC5883L datasheets don't specify behaviour if only vcc_io is powered / if I2C is pulled to VCC while chip is powered down
Connections:
- net labels removed: VCC
- wire segments 33 -> 34
Changed lines of the file:
@@
 Sheet 2 2
 Title "Sensors"
-Date "11 feb 2014"
+Date "13 feb 2014"
 Rev ""
 Comp ""
@@
 Text HLabel 2250 1650 0    60   Input ~ 0
 VCC_A
-Text HLabel 7250 1700 0    60   Input ~ 0
-VCC
 $Comp
 L _MPU6000 U9
@@
 $EndComp
 $Comp
-L GND #PWR055
+L GND #PWR052
 U 1 1 518B161E
 P 2450 4250
-F 0 "#PWR055" H 2450 4250 30  0001 C CNN
+F 0 "#PWR052" H 2450 4250 30  0001 C CNN
 F 1 "GND" H 2450 4180 30  0001 C CNN
 F 2 "" H 2450 4250 60  0001 C CNN
@@
 $EndComp
 $Comp
-L GND #PWR056
+L GND #PWR053
 U 1 1 518B161C
 P 1400 4550
-F 0 "#PWR056" H 1400 4550 30  0001 C CNN
+F 0 "#PWR053" H 1400 4550 30  0001 C CNN
 F 1 "GND" H 1400 4480 30  0001 C CNN
 F 2 "" H 1400 4550 60  0001 C CNN
@@
 $EndComp
 $Comp
-L GND #PWR057
+L GND #PWR054
 U 1 1 518B161B
 P 2100 4950
-F 0 "#PWR057" H 2100 4950 30  0001 C CNN
+F 0 "#PWR054" H 2100 4950 30  0001 C CNN
 F 1 "GND" H 2100 4880 30  0001 C CNN
 F 2 "" H 2100 4950 60  0001 C CNN
@@
 $EndComp
 $Comp
-L GND #PWR058
+L GND #PWR055
 U 1 1 518B1619
 P 2450 5050
-F 0 "#PWR058" H 2450 5050 30  0001 C CNN
+F 0 "#PWR055" H 2450 5050 30  0001 C CNN
 F 1 "GND" H 2450 4980 30  0001 C CNN
 F 2 "" H 2450 5050 60  0001 C CNN
@@
 $EndComp
 $Comp
-L GND #PWR059
+L GND #PWR056
 U 1 1 518B1613
 P 7250 2200
-F 0 "#PWR059" H 7250 2200 30  0001 C CNN
+F 0 "#PWR056" H 7250 2200 30  0001 C CNN
 F 1 "GND" H 7250 2130 30  0001 C CNN
 F 2 "" H 7250 2200 60  0001 C CNN
@@
 $EndComp
 $Comp
-L GND #PWR060
+L GND #PWR057
 U 1 1 518B1610
 P 8800 2600
-F 0 "#PWR060" H 8800 2600 30  0001 C CNN
+F 0 "#PWR057" H 8800 2600 30  0001 C CNN
 F 1 "GND" H 8800 2530 30  0001 C CNN
 F 2 "" H 8800 2600 60  0001 C CNN
@@
 NoConn ~ 3900 1850
 $Comp
-L GND #PWR061
+L GND #PWR058
 U 1 1 518B160E
 P 3900 2100
-F 0 "#PWR061" H 3900 2100 30  0001 C CNN
+F 0 "#PWR058" H 3900 2100 30  0001 C CNN
 F 1 "GND" H 3900 2030 30  0001 C CNN
 F 2 "" H 3900 2100 60  0001 C CNN
@@
 $EndComp
 $Comp
-L GND #PWR062
+L GND #PWR059
 U 1 1 518B160D
 P 2300 2150
-F 0 "#PWR062" H 2300 2150 30  0001 C CNN
+F 0 "#PWR059" H 2300 2150 30  0001 C CNN
 F 1 "GND" H 2300 2080 30  0001 C CNN
 F 2 "" H 2300 2150 60  0001 C CNN
@@
 Connection ~ 7250 4250
 $Comp
-L GND #PWR063
+L GND #PWR060
 U 1 1 5196E087
 P 7150 4800
-F 0 "#PWR063" H 7150 4800 30  0001 C CNN
+F 0 "#PWR060" H 7150 4800 30  0001 C CNN
 F 1 "GND" H 7150 4730 30  0001 C CNN
 F 2 "" H 7150 4800 60  0000 C CNN
@@
 $EndComp
 $Comp
-L GND #PWR064
+L GND #PWR061
 U 1 1 5196E096
 P 8400 5250
-F 0 "#PWR064" H 8400 5250 30  0001 C CNN
+F 0 "#PWR061" H 8400 5250 30  0001 C CNN
 F 1 "GND" H 8400 5180 30  0001 C CNN
 F 2 "" H 8400 5250 60  0000 C CNN
@@
 Connection ~ 8400 5150
 $Comp
-L GND #PWR065
+L GND #PWR062
 U 1 1 5196E151
 P 7700 4700
-F 0 "#PWR065" H 7700 4700 30  0001 C CNN
+F 0 "#PWR062" H 7700 4700 30  0001 C CNN
 F 1 "GND" H 7700 4630 30  0001 C CNN
 F 2 "" H 7700 4700 60  0000 C CNN
@@
 	1    0    0    -1
 $EndComp
-Text HLabel 9100 4700 2    60   Input ~ 0
-VCC
-Text HLabel 7700 4350 0    60   Input ~ 0
-VCC
-Text HLabel 7700 4600 0    60   Input ~ 0
-VCC
-Text HLabel 9100 4800 2    60   Input ~ 0
-VCC
 Text HLabel 9100 4400 2    60   BiDi ~ 0
 I2C_SDA
@@
 	7150 4750 7150 4800
 Connection ~ 7150 4750
+Text HLabel 7700 4600 0    60   Input ~ 0
+VCC_A
+Wire Wire Line
+	7250 1700 7250 1600
+Connection ~ 7250 1600
+Text HLabel 7700 4350 0    60   Input ~ 0
+VCC_A
+Text HLabel 9100 4700 2    60   Input ~ 0
+VCC_A
+Text HLabel 9100 4800 2    60   Input ~ 0
+VCC_A
 $EndSCHEMATC

Commit message: updated library, changed component names according to new lib
This fixes the library editor problem, where components disappear.
Parts:
- U10: symbol _HMC5883L -> HMC5883L
- U11: symbol _H3LIS331DL -> H3LIS331DL
- U8: symbol _MS5611-01BA -> MS5611-01BA
- U9: symbol _MPU6000 -> MPU6000
Changed lines of the file:
@@
 VCC_A
 $Comp
-L _MPU6000 U9
+L MPU6000 U9
 U 1 1 518B161F
 P 3600 4550
@@
 NoConn ~ 2650 4900
 $Comp
-L _HMC5883L U10
+L HMC5883L U10
 U 1 1 518B1617
 P 8250 1800
@@
 $EndComp
 $Comp
-L _MS5611-01BA U8
+L MS5611-01BA U8
 U 1 1 518B160F
 P 3150 1850
@@
 $EndComp
 $Comp
-L _H3LIS331DL U11
+L H3LIS331DL U11
 U 1 1 5196DFD7
 P 8400 4600
